File: Sienkiewicz_TOUCH.kicad_pcb (KiCad board)
At the start: 6 copper layers, 0 parts

Commit message: sienkiewicz library missing value update
Parts:
- added D1: RED, Diode_SMD:D_1206_3216Metric, F.Cu at (165.5, 97.0)
- added D2: RED, Diode_SMD:D_1206_3216Metric, F.Cu at (165.5, 83.0)
- added J1: Conn_ARM_SWD_TagConnect_TC2030-NL, Connector:Tag-Connect_TC2030-IDC-NL_2x03_P1.27mm_Vertical, F.Cu at (148.5, 105.6)
- added R1: 1k, Resistor_SMD:R_0805_2012Metric, F.Cu at (153.5, 97.0)
- added R2: 1k, Resistor_SMD:R_0805_2012Metric, F.Cu at (143.6, 97.0)
- added Rd1: 5k1, Resistor_SMD:R_0805_2012Metric, F.Cu at (140.5, 73.0)
- added Rd2: 5k1, Resistor_SMD:R_0805_2012Metric, F.Cu at (156.5, 73.0)
- added U1: ATtiny204-SS, Package_SO:SOIC-14_3.9x8.7mm_P1.27mm, F.Cu at (162.0, 90.0)
- added U2: ~, __Sienkiewicz:Sienkiewicz, F.Cu at (148.5, 90.0)
Other:
- board outline added: 38 x 38 mm
