File: Revision History.kicad_sch (KiCad schematic)
At the start: 0 parts

Commit message: prep for 2.0.2 release
Changed lines of the file:
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@@
 		)
 	)
-	(text_box "${RELEASE_TITLE_1.0.2}"
+	(text_box "${RELEASE_TITLE_2.0.2}"
 		(exclude_from_sim no)
-		(at 152.4 31.75 0)
+		(at 20.32 88.9 0)
 		(size 57.15 7.62)
 		(margins 1.4287 1.4287 1.4287 1.4287)
@@
 		)
 	)
-	(text_box "${RELEASE_BODY_1.0.2}"
+	(text_box "${RELEASE_BODY_2.0.2}"
 		(exclude_from_sim no)
-		(at 154.94 35.56 0)
-		(size 58.42 111.76)
+		(at 22.86 93.98 0)
+		(size 58.42 93.98)
 		(margins 1.4287 1.4287 1.4287 1.4287)
 		(stroke
@@
 		(exclude_from_sim no)
 		(at 22.86 63.5 0)
-		(size 123.19 77.47)
+		(size 60.96 22.86)
 		(margins 1.4287 1.4287 1.4287 1.4287)
 		(stroke
