File: Revision History.kicad_sch (KiCad schematic)
At the start: 0 parts

Commit message: documentation update /requirements /schematic
Changed lines of the file:
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@@
+		)
+	)
+	(text_box "${RELEASE_BODY_2.1.1}"
+		(exclude_from_sim no)
+		(at 88.9 34.29 0)
+		(size 58.42 35.56)
+		(margins 1.4287 1.4287 1.4287 1.4287)
+		(stroke
+			(width -0.0001)
+			(type default)
+		)
+		(fill
+			(type none)
+		)
+		(effects
+			(font
+				(face "Arial")
+				(size 1.905 1.905)
+				(color 0 0 0 1)
+			)
+			(justify left top)
 		)
 	)
@@
 		)
 	)
+	(text_box "${RELEASE_TITLE_2.1.1}"
+		(exclude_from_sim no)
+		(at 86.36 31.75 0)
+		(size 57.15 7.62)
+		(margins 1.4287 1.4287 1.4287 1.4287)
+		(stroke
+			(width -0.0001)
+			(type solid)
+		)
+		(fill
+			(type none)
+		)
+		(effects
+			(font
+				(face "Arial")
+				(size 1.905 1.905)
+				(thickness 0.254)
+				(bold yes)
+			)
+			(justify left top)
+		)
+	)
 	(text_box "${RELEASE_BODY_2.1.0}"
 		(exclude_from_sim no)
 		(at 22.86 121.92 0)
-		(size 58.42 71.12)
+		(size 58.42 35.56)
 		(margins 1.4287 1.4287 1.4287 1.4287)
 		(stroke
