File: Section B - uC.kicad_sch (KiCad schematic)
At the start: 9 parts, among them J1 TC2030-NL, U1 ATtiny204-SS

Commit message: routing update #4
Connections:
- net SR_SDI is gone; now on net SR_CLK: U1.11 (PA1)
- net SR_CLK: no longer U1.9 (PB0)
- new net SR_DAT: U1.9 (PB0)
Changed lines of the file:
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@@
 		)
 	)
-	(label "SR_SDI"
+	(label "SR_CLK"
 		(at 153.67 77.47 180)
 		(effects
@@
 		)
 	)
-	(label "SR_CLK"
+	(label "SR_DAT"
 		(at 107.95 74.93 0)
 		(effects
@@
 		)
 	)
-	(hierarchical_label "SR_CLK"
+	(hierarchical_label "SR_DAT"
 		(shape output)
 		(at 105.41 74.93 180)
@@
 		)
 	)
-	(hierarchical_label "SR_SDI"
+	(hierarchical_label "SR_CLK"
 		(shape output)
 		(at 156.21 77.47 0)
