File: Section D - Shift Register screw interface.kicad_sch (KiCad schematic)
At the start: 1 part

Commit message: routing update #4
Connections:
- net SR_SDI is gone; now on net SR_CLK: B1.1 (CLK)
- net SR_CLK: no longer B1.4 (CLK)
- new net SR_DAT: B1.4 (DAT)
Changed lines of the file:
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@@
+	(wire
+		(pts
+			(xy 129.54 88.9) (xy 132.08 88.9)
+		)
+		(stroke
+			(width 0)
+			(type default)
+		)
+	)
 	(wire
 		(pts
 			(xy 144.78 101.6) (xy 170.18 101.6)
+		)
+		(stroke
+			(width 0)
+			(type default)
+		)
+	)
+	(wire
+		(pts
+			(xy 129.54 83.82) (xy 132.08 83.82)
 		)
 		(stroke
@@
 		)
 	)
-	(hierarchical_label "SR_SDI"
+	(hierarchical_label "SR_DAT"
 		(shape input)
-		(at 132.08 83.82 180)
+		(at 129.54 88.9 180)
 		(effects
 			(font
@@
 	(hierarchical_label "SR_CLK"
 		(shape input)
-		(at 132.08 88.9 180)
+		(at 129.54 83.82 180)
 		(effects
 			(font
